File: hardware/pcb/vbt_v1_schematic/vbt_v1_schematic.kicad_sch (KiCad schematic)
At the start: 0 parts

Commit message: fix: added logic so that reps are only detected on ascent. In the future, I may change so that it can measure both, or one or the other. For now, it is only the ascent.
Parts:
- added R1, R2: R, symbol Device:R
- added U1: (no value), ESP32_30pin, symbol esp32_30pin_revised:ESP32_30Pin
- added U2: INA240A1PW, Package_SO:TSSOP-8_4.4x3mm_P0.65mm, symbol Amplifier_Current:INA240A1PW
- added U3: SN74LVC2G14DBV, Package_TO_SOT_SMD:SOT-23-6, symbol 74xGxx:SN74LVC2G14DBV
- added U4: ZXCT1009F, Package_TO_SOT_SMD:SOT-23, symbol Amplifier_Current:ZXCT1009F
Connections:
- new net: R1.1, R2.1, U1.16 (3.3v)
- new net: U2.1 (GND), U2.4 (GND)
- new net DSI_SCL: U1.29 (GPIO22)
- new net DSI_SDA: U1.26 (GPIO21)
- new net ENC_A: R1.2, U1.24 (GPIO18)
- new net ENC_B: R2.2, U1.25 (GPIO19)

Commit message: pcb_v1_updates
Parts:
- removed U2: INA240A1PW, Package_SO:TSSOP-8_4.4x3mm_P0.65mm, symbol Amplifier_Current:INA240A1PW
- removed U3: SN74LVC2G14DBV, Package_TO_SOT_SMD:SOT-23-6, symbol 74xGxx:SN74LVC2G14DBV
- removed U4: ZXCT1009F, Package_TO_SOT_SMD:SOT-23, symbol Amplifier_Current:ZXCT1009F
- added BT1: 18650 protected, symbol Device:Battery_Cell
- added DISP1: OLED DISP, symbol Connector_Generic:Conn_01x04
- added ENC1: Encoder, symbol Connector_Generic:Conn_01x04
- added F1: PTC 1.5A, symbol Device:Fuse
- added Q1: AO3401A, Package_TO_SOT_SMD:SOT-23, symbol Transistor_FET:AO3401A
- added SW1, SW2: SW_SPST, symbol Switch:SW_SPST
- R3: renamed from R2; value R -> 10 kOhm
- R4: renamed from R1; value R -> 10 kOhm
- U3: renamed from U1; footprint ESP32_30pin -> ESP32 DevKit v1
Connections:
- net ENC_A: now also ENC1.4 (Pin_4)
- net ENC_B: now also ENC1.3 (Pin_3)
- net GND: now reaches U3.17 (GND)
- net GND: now also DISP1.2 (Pin_2), ENC1.1 (Pin_1)
- net at U3.2 (GND): now also BT1.2 (-), Q1.1 (G), SW2.2 (B)
- net at U3.20 (GPIO4): now also SW2.1 (A)
- net DSI_SCL renamed OLED_SCL
- net OLED_SCL: now also DISP1.3 (Pin_3)
- net DSI_SDA renamed OLED_SDA
- net OLED_SDA: now also DISP1.4 (Pin_4)
- new net: F1.2, SW1.1 (A)
- new net: F1.1, Q1.2 (S)
- new net: BT1.1 (+), Q1.3 (D)
- new net +3.3V: DISP1.1 (Pin_1)
- new net +5V: ENC1.2 (Pin_2)
- no-connect marks 0 -> 21
Other:
- moved on the sheet: R3, R4, U3

Commit message: update: pcb layout complete
Parts:
- added U2: Conn_01x04, Connector_PinHeader_2.54mm:PinHeader_1x04_P2.54mm_Vertical, symbol Connector_Generic:Conn_01x04
- DISP1: footprint (none) -> Connector_PinSocket_2.54mm:PinSocket_1x04_P2.54mm_Vertical
- ENC1: footprint (none) -> Connector_PinHeader_2.54mm:PinHeader_1x04_P2.54mm_Vertical
- F1: footprint (none) -> Fuse:Fuse_1812_4532Metric_Pad1.30x3.40mm_HandSolder
- R3, R4: value 10 kOhm -> 10kΩ; footprint (none) -> Resistor_THT:R_Axial_DIN0207_L6.3mm_D2.5mm_P10.16mm_Horizontal
- SW1: footprint (none) -> Connector_PinHeader_2.54mm:PinHeader_1x02_P2.54mm_Vertical
- SW2: footprint (none) -> Button_Switch_THT:SW_PUSH_6mm
Connections:
- net +3.3V is gone; now on an unnamed net: DISP1.1 (Pin_1)
- net +5V: now also U3.1 (VIN), U2.1 (Pin_1)
- net GND: now also BT1.2 (-), SW2.2 (B), U2.2 (Pin_2)
- net at SW1.1 (A): now also U2.3 (Pin_3); no longer F1.2
- net at SW1.2 (B): now also F1.2
- net at Q1.1 (G), U3.2 (GND): no longer BT1.2 (-), SW2.2 (B)
- no-connect marks 21 -> 22
Other:
- note added: "DISPLAY"
- note added: "ENCODER"
- note added: "GND"
- note added: "POWER"
- note added: "VIN"
- note added: "VOUT"
- title: (none) -> VBT WIRING V1
- moved on the sheet: BT1, DISP1, ENC1, F1, Q1, R3, R4, SW1, SW2, U3
