File: hardware/pcb/v2_kicad/offboard_power_wiring.kicad_sch (KiCad schematic)
At the start: 5 parts, among them J5 TP4056 USB-C with Protection, J6 5V boost, J7 3.3V buck-boost, SW3 Slide Switch

Commit message: Updated Schematic
Parts:
- added F1: Polyfuse, symbol Device:Polyfuse
- added Q1: AO3401A, Package_TO_SOT_SMD:SOT-23, symbol Transistor_FET:AO3401A
- added R9: 10k, Resistor_SMD:R_0805_2012Metric, symbol Device:R
Connections:
- net B+: now also F1.1, Q1.2 (S)
- net B-: now also R9.2
- new net: F1.2, Q1.3 (D)
- new net: Q1.1 (G), R9.1
Other:
- moved on the sheet: BT1

Commit message: updated pcb schematic for finalized BOM
Parts:
- F1: footprint (none) -> Fuse:Fuse_1206_3216Metric
Changed lines of the file:
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@@
 		(exclude_from_sim no)
 		(in_bom yes)
-		(on_board yes)
+		(on_board no)
 		(in_pos_files yes)
 		(dnp no)
@@
 			)
 		)
-		(property "Footprint" ""
+		(property "Footprint" "Fuse:Fuse_1206_3216Metric"
 			(at 96.52 62.23 0)
 			(hide yes)
@@
 		(exclude_from_sim no)
 		(in_bom yes)
-		(on_board yes)
+		(on_board no)
 		(in_pos_files yes)
 		(dnp no)
@@
 		(exclude_from_sim no)
 		(in_bom yes)
-		(on_board yes)
+		(on_board no)
 		(in_pos_files yes)
 		(dnp no)
@@
 		(exclude_from_sim no)
 		(in_bom yes)
-		(on_board yes)
-		(in_pos_files yes)
-		(dnp no)
+		(on_board no)
+		(in_pos_files yes)
+		(dnp no)
