File: hardware/pcb/v2_kicad/vbt_kicad_pcb.kicad_pcb (KiCad board)
At the start: 2 copper layers, 70 x 50 mm, 18 parts, among them J1 Conn_01x03, J2 Conn_01x04, J3 Conn_01x04, J4 Conn_01x04, SW1 SW_Push, SW2 SW_Push, U1 ESP32-WROOM-32E

Commit message: updated pcb schematic for finalized BOM
Parts:
- added C5: 100nF, Capacitor_SMD:C_0805_2012Metric_Pad1.18x1.45mm_HandSolder, F.Cu at (167.9, 61.3)
- added D1: LED, LED_THT:LED_D5.0mm, F.Cu at (154.5, 63.0)
- added J8: Conn_01x04, Connector_JST:JST_XH_B4B-XH-A_1x04_P2.50mm_Vertical, F.Cu at (161.5, 55.3)
- added R8: 330Ω, Resistor_SMD:R_0805_2012Metric, F.Cu at (167.7, 64.2)
- J1: footprint Connector_PinSocket_2.54mm:PinSocket_1x03_P2.54mm_Vertical -> Connector_JST:JST_XH_B3B-XH-A_1x03_P2.50mm_Vertical
- J2: value Conn_01x04 -> Conn_01x05; footprint Connector:FanPinHeader_1x04_P2.54mm_Vertical -> Connector_JST:JST_XH_B5B-XH-A_1x05_P2.50mm_Vertical
- J3, J4: footprint Connector:FanPinHeader_1x04_P2.54mm_Vertical -> Connector_JST:JST_XH_B4B-XH-A_1x04_P2.50mm_Vertical
- R1, R2: value R -> 10k
- R6, R7: footprint Resistor_SMD:R_0805_2012Metric_Pad1.20x1.40mm_HandSolder -> Resistor_SMD:R_0805_2012Metric
- SW1, SW2: footprint Inductor_SMD:L_0805_2012Metric -> VBT_parts:SW_Tactile_SCHURTER_LSH_6x6mm
Connections:
- C1 pad 2: GND -> Net-(J1-Pin_3)
- C2 pad 2: GND -> Net-(J1-Pin_3)
- C3 pad 2: GND -> Net-(J1-Pin_3)
- J1 pad 1: GND -> /ESP_TX
- J1 pad 2: /ESP_TX -> /ESP_RX
- J1 pad 3: /ESP_RX -> Net-(J1-Pin_3)
- J2 pad 1: GND -> /ENC_A
- J2 pad 2: /+5V -> /ENC_B
- J2 pad 3: /ENC_B -> +3V3
- J2 pad 4: /ENC_A -> GND
- J3 pad 1: GND -> /I2C_SCL
- J3 pad 2: +3V3 -> /I2C_SDA
- J3 pad 3: /I2C_SDA -> +3V3
- J3 pad 4: /I2C_SCL -> GND
- J4 pad 1: /+5V -> +3V3
- J4 pad 3: Net-(J4-Pin_3) -> VBAT
- R6 pad 1: Net-(J4-Pin_3) -> VBAT
- R7 pad 1: GND -> Net-(J1-Pin_3)
- R7 pad 2: Net-(J4-Pin_3) -> /VBAT_SENSE
- SW1 pad 1: GND -> Net-(J1-Pin_3)
- SW2 pad 1: GND -> Net-(J1-Pin_3)
- SW2 pad 2: GND -> Net-(U1-IO0)
- U1 pad 25: GND -> Net-(U1-IO0)
- U1 pad 26: /LED -> Net-(U1-IO4)
- U1 pad 34: unconnected-(U1-RXD0/IO3-Pad34) -> /ESP_RX
- U1 pad 35: unconnected-(U1-TXD0/IO1-Pad35) -> /ESP_TX

Commit message: updated pcb layout
Parts:
- removed C4: 1 µF, Capacitor_SMD:C_0805_2012Metric
- J1: value Conn_01x03 -> Serial Connector
- J2: value Conn_01x05 -> Rotary Encoder
- J3: value Conn_01x04 -> I2C Display
- J4: value Conn_01x04 -> Power Connector
- J8: value Conn_01x04 -> I2C Magnet Sensor
- moved C5 54.3 mm to (125.0, 94.5)
- moved J4 46.1 mm to (138.0, 98.0), turned to 180 degrees
- moved R6 35.8 mm to (125.0, 87.0), turned to 180 degrees
- moved R7 35.3 mm to (125.0, 89.0), turned to 180 degrees
- moved R5 27.6 mm to (120.0, 62.9), turned to -90 degrees
- moved R8 25.9 mm to (141.9, 62.5), turned to 180 degrees
- moved R3 24.3 mm to (126.0, 62.9), turned to -90 degrees
- moved R4 23.0 mm to (123.5, 62.9), turned to -90 degrees
- moved SW2 21.8 mm to (145.4, 89.2)
- moved SW1 14.3 mm to (145.4, 81.2)
- moved D1 13.6 mm to (142.5, 69.5)
- moved R2 12.1 mm to (129.0, 62.9), turned to -90 degrees
- moved J1 11.6 mm to (151.0, 97.0), turned to 0 degrees
- moved J8 7.90 mm to (156.0, 61.0), turned to -90 degrees
- moved J2 6.95 mm to (120.0, 54.0)
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Connections:
- C1 pad 2: Net-(J1-Pin_3) -> GND
- C2 pad 2: Net-(J1-Pin_3) -> GND
- C3 pad 2: Net-(J1-Pin_3) -> GND
- C5 pad 2: Net-(J1-Pin_3) -> GND
- J1 pad 3: Net-(J1-Pin_3) -> GND
- R7 pad 1: Net-(J1-Pin_3) -> GND
- SW1 pad 1: Net-(J1-Pin_3) -> GND
- SW2 pad 1: Net-(J1-Pin_3) -> GND
Routing:
- net GND: track 128.7 -> 39.1 mm
- net /ESP_RX: track 0.00 -> 14.0 mm
Other:
- board size 70 x 50 mm -> 70 x 70 mm
