File: hardware/pcb/v2_kicad/vbt_kicad_pcb.kicad_pcb (KiCad board)
At the start: 2 copper layers, 70 x 70 mm, 21 parts, among them J1 Serial Connector, J2 Rotary Encoder, J3 I2C Display, J4 Power Connector, J8 I2C Magnet Sensor, SW1 SW_Push, SW2 SW_Push, U1 ESP32-WROOM-32E

Commit message: added reset button connector to diagram and pcb layout
Parts:
- added J9: Rep Reset Button, Connector_JST:JST_XH_B2B-XH-A_1x02_P2.50mm_Vertical, F.Cu at (156.0, 75.0)
Connections:
- U1 pad 16: unconnected-(U1-IO13-Pad16) -> Net-(J9-Pin_2)

Commit message: updated pcb
Parts:
- moved J2 37.2 mm to (156.0, 63.5), turned to -90 degrees
- moved J8 21.2 mm to (136.0, 54.0), turned to 0 degrees
- moved J3 14.5 mm to (121.5, 54.0)
- moved SW2 11.3 mm to (145.0, 78.0)
- moved J9 5.50 mm to (156.0, 80.5)
- moved SW1 5.27 mm to (145.0, 86.5), turned to 0 degrees
Routing:
- net /ENC_A: track 0.00 -> 37.0 mm
- net /ENC_B: track 0.00 -> 30.9 mm
- net /I2C_SDA: track 0.00 -> 29.4 mm
- net /I2C_SCL: track 0.00 -> 29.3 mm
- net GND: track 39.1 -> 12.5 mm
- net +3V3: track 0.00 -> 25.9 mm
- net Net-(U1-EN): track 19.1 -> 39.4 mm
- net /ESP_RX: track 14.0 -> 0.00 mm
- net VBAT: track 0.00 -> 13.9 mm
- net Net-(U1-IO0): track 0.00 -> 11.6 mm
